File: writerdeck-pcbs/writerdeck-pcbs.kicad_pcb (KiCad board)
At the start: 2 copper layers, 1 x 0.7 mm, 5 parts, among them J1 USB_C_Receptacle, J2 12401826E412A, U1 RP2040, U2 BQ25792RQMR

Commit message: power management done
Parts:
- added C1: 10u, Capacitor_SMD:C_0603_1608Metric, F.Cu at (74.4, 17.5)
- added C10: 10u, Capacitor_SMD:C_0603_1608Metric, F.Cu at (78.4, 17.5)
- added C11: 10u, Capacitor_SMD:C_0603_1608Metric, F.Cu at (78.4, 20.0)
- added C12: 47n, Capacitor_SMD:C_0603_1608Metric, F.Cu at (78.4, 22.5)
- added C13: 47n, Capacitor_SMD:C_0603_1608Metric, F.Cu at (78.4, 25.0)
- added C14: 100n, Capacitor_SMD:C_0603_1608Metric, F.Cu at (78.4, 27.5)
- added C15: 10u, Capacitor_SMD:C_0603_1608Metric, F.Cu at (78.4, 30.1)
- added C16: 10u, Capacitor_SMD:C_0603_1608Metric, F.Cu at (78.4, 32.6)
- added C17: 10u, Capacitor_SMD:C_0603_1608Metric, F.Cu at (78.4, 35.1)
- added C18: 10u, Capacitor_SMD:C_0603_1608Metric, F.Cu at (78.4, 37.6)
- added C19: 10u, Capacitor_SMD:C_0603_1608Metric, F.Cu at (82.4, 17.5)
- added C2: 22u, Capacitor_SMD:C_0603_1608Metric, F.Cu at (74.4, 20.0)
- added C20: 10u, Capacitor_SMD:C_0603_1608Metric, F.Cu at (82.4, 20.0)
- added C21: 100n, Capacitor_SMD:C_0603_1608Metric, F.Cu at (74.2, 48.8)
- added C23: 10u, Capacitor_SMD:C_0603_1608Metric, F.Cu at (82.4, 22.5)
- added C24: 22u, Capacitor_SMD:C_0603_1608Metric, F.Cu at (82.4, 25.0)
- added C25: 22u, Capacitor_SMD:C_0603_1608Metric, F.Cu at (82.4, 27.5)
- added C26: 100n, Capacitor_SMD:C_0603_1608Metric, F.Cu at (74.2, 51.3)
- added C3: 4u7, Capacitor_SMD:C_0603_1608Metric, F.Cu at (74.4, 22.5)
- added C4: 100n, Capacitor_SMD:C_0603_1608Metric, F.Cu at (74.4, 25.0)
- added C5: 10u, Capacitor_SMD:C_0603_1608Metric, F.Cu at (74.4, 27.5)
- added C6: 10u, Capacitor_SMD:C_0603_1608Metric, F.Cu at (74.4, 30.1)
- added C7: 2u2, Capacitor_SMD:C_0603_1608Metric, F.Cu at (74.4, 32.6)
- added C8: 100n, Capacitor_SMD:C_0603_1608Metric, F.Cu at (74.4, 35.1)
- added C9: 10u, Capacitor_SMD:C_0603_1608Metric, F.Cu at (74.4, 37.6)
- added D1: Blue LED, LED_SMD:LED_0805_2012Metric, F.Cu at (65.5, 40.8)
- added D2: Red LED, LED_SMD:LED_0805_2012Metric, F.Cu at (80.4, 49.1)
- added D3: Green LED, LED_SMD:LED_0805_2012Metric, F.Cu at (80.4, 52.1)
- added J12401826E412A1: USB_C_Receptacle, ZF_common:12401826E412A, F.Cu at (63.1, 53.5)
- added L2: 1u, ZF_common:XFL4020-102MEC, F.Cu at (60.3, 42.2)
- added Q1: CSD17575Q3, Package_TO_SOT_SMD:TDSON-8-1, F.Cu at (76.5, 42.2)
- added R1: 2, Resistor_SMD:R_0603_1608Metric, F.Cu at (82.4, 30.1)
- added R10: 10k, Resistor_SMD:R_0603_1608Metric, F.Cu at (86.4, 27.5)
- added R11: 2k2, Resistor_SMD:R_0603_1608Metric, F.Cu at (74.2, 53.8)
- added R12: 100, Resistor_SMD:R_0603_1608Metric, F.Cu at (86.4, 30.1)
- added R13: 10k, Resistor_SMD:R_0603_1608Metric, F.Cu at (86.4, 32.6)
- added R14: 100k, Resistor_SMD:R_0603_1608Metric, F.Cu at (86.4, 35.1)
- added R15: 1k, Resistor_SMD:R_0603_1608Metric, F.Cu at (84.6, 48.8)
- added R16: 1k, Resistor_SMD:R_0603_1608Metric, F.Cu at (84.6, 51.3)
- added R17: 10k, Resistor_SMD:R_0603_1608Metric, F.Cu at (86.4, 37.6)
- added R18: 100k, Resistor_SMD:R_0603_1608Metric, F.Cu at (90.4, 17.5)
- added R19: 732k, Resistor_SMD:R_0603_1608Metric, F.Cu at (90.4, 20.0)
- added R2: 10k, Resistor_SMD:R_0603_1608Metric, F.Cu at (82.4, 32.6)
- added R20: 620, Resistor_SMD:R_0603_1608Metric, F.Cu at (90.4, 22.5)
- added R24: 15k, Resistor_SMD:R_0603_1608Metric, F.Cu at (90.4, 25.0)
- added R25: 100, Resistor_SMD:R_0603_1608Metric, F.Cu at (90.4, 27.5)
- added R26: 50, Resistor_SMD:R_0603_1608Metric, F.Cu at (90.4, 30.1)
- added R3: 3k, Resistor_SMD:R_0603_1608Metric, F.Cu at (82.4, 35.1)
- added R4: 10k, Resistor_SMD:R_0603_1608Metric, F.Cu at (82.4, 37.6)
- added R5: 300k, Resistor_SMD:R_0603_1608Metric, F.Cu at (86.4, 17.5)
- added R6: 2k2, Resistor_SMD:R_0603_1608Metric, F.Cu at (86.4, 20.0)
- added R8: 2k, Resistor_SMD:R_0603_1608Metric, F.Cu at (86.4, 22.5)
- added R9: 10k, Resistor_SMD:R_0603_1608Metric, F.Cu at (86.4, 25.0)
- added U4: TPS61022, Package_DFN_QFN:Texas_RWU0007A_VQFN-7_2x2mm_P0.5mm, F.Cu at (69.9, 41.0)
- J1: value USB_C_Receptacle -> 5023520300; footprint Connector_USB:USB_C_Receptacle_GCT_USB4110 -> ZF_common:5023520300
- J2: value 12401826E412A -> 5023520300; footprint ZF_common:12401826E412A -> ZF_common:5023520300
- moved U2 28.9 mm to (84.3, 41.8)
- moved J1 28.2 mm to (66.1, 22.2)
- moved Module1 19.0 mm to (18.3, 68.3)
- moved U1 15.2 mm to (62.1, 66.9)
- moved J2 10.3 mm to (66.1, 33.7)
Connections:
- Module1 pad 21: unconnected-(Module1A-LED_nACT-Pad21) -> /Base/CM5 GPIO/LED_nACT
- Module1 pad 92: unconnected-(Module1A-PWR_BUT-Pad92) -> PWR_BUT
- Module1 pad 95: unconnected-(Module1A-LED_nPWR-Pad95) -> /Base/CM5 GPIO/LED_nPWR
- U2 pad 1: unconnected-(U2-STAT-Pad1) -> /Base/Power Management/STAT
- U2 pad 10: unconnected-(U2-ACDRV2-Pad10) -> GND
- U2 pad 11: unconnected-(U2-ACDRV1-Pad11) -> GND
- U2 pad 12: unconnected-(U2-~{QON}-Pad12) -> PWR_BUT
- U2 pad 13: unconnected-(U2-~{CE}-Pad13) -> Net-(U2-~{CE})
- U2 pad 14: unconnected-(U2-SCL-Pad14) -> Net-(U2-SCL)
- U2 pad 15: unconnected-(U2-SDA-Pad15) -> Net-(U2-SDA)
- U2 pad 16: unconnected-(U2-TS-Pad16) -> /Base/Power Management/BATT_TEMP
- U2 pad 17: unconnected-(U2-ILIM_HIZ-Pad17) -> /Base/Power Management/ILIM_HIZ
- U2 pad 18: unconnected-(U2-BATP-Pad18) -> /Base/Power Management/BATP
- U2 pad 19: unconnected-(U2-BTST2-Pad19) -> /Base/Power Management/BTST2
- U2 pad 2: unconnected-(U2-VBUS-Pad2) -> VBUS
- U2 pad 20: unconnected-(U2-PROG-Pad20) -> Net-(U2-PROG)
- U2 pad 21: unconnected-(U2-~{INT}-Pad21) -> Net-(U2-~{INT})
- U2 pad 22: unconnected-(U2-BAT-Pad22) -> /Base/Power Management/BAT
- U2 pad 23: unconnected-(U2-BAT__1-Pad23) -> /Base/Power Management/BAT
- U2 pad 24: unconnected-(U2-SDRV-Pad24) -> /Base/Power Management/SDRV
- U2 pad 25: unconnected-(U2-SYS-Pad25) -> /Base/Power Management/VSYS
- U2 pad 26: unconnected-(U2-SW2-Pad26) -> /Base/Power Management/SW2
- U2 pad 27: unconnected-(U2-GND-Pad27) -> GND
- U2 pad 28: unconnected-(U2-SW1-Pad28) -> /Base/Power Management/SW1
- U2 pad 29: unconnected-(U2-PMID-Pad29) -> Net-(U2-PMID)
- U2 pad 3: unconnected-(U2-VBUS__1-Pad3) -> VBUS
- U2 pad 4: unconnected-(U2-BTST1-Pad4) -> /Base/Power Management/BTST1
- U2 pad 5: unconnected-(U2-REGN-Pad5) -> /Base/Power Management/REGN
- U2 pad 6: /Base/Power Management/USB2_P -> /Base/USB2_P
- U2 pad 7: /Base/Power Management/USB2_N -> /Base/USB2_N
- U2 pad 8: unconnected-(U2-VAC2-Pad8) -> VBUS
- U2 pad 9: unconnected-(U2-VAC1-Pad9) -> VBUS

Commit message: backup
Parts:
- removed R26: 50, Resistor_SMD:R_0603_1608Metric
- added C22: 4u7, Capacitor_SMD:C_0603_1608Metric, F.Cu at (87.5, 58.2)
- added C28: 22p, Capacitor_SMD:C_0603_1608Metric, F.Cu at (93.5, 19.2)
- added C29: 1u, Capacitor_SMD:C_0603_1608Metric, F.Cu at (93.5, 21.7)
- added C30: 22p, Capacitor_SMD:C_0603_1608Metric, F.Cu at (93.5, 24.2)
- added C31: 100n, Capacitor_SMD:C_0603_1608Metric, F.Cu at (93.5, 26.7)
- added C32: 100n, Capacitor_SMD:C_0603_1608Metric, F.Cu at (93.5, 29.2)
- added C33: 100n, Capacitor_SMD:C_0603_1608Metric, F.Cu at (97.5, 16.7)
- added C34: 100n, Capacitor_SMD:C_0603_1608Metric, F.Cu at (97.5, 19.2)
- added C35: 1u, Capacitor_SMD:C_0603_1608Metric, F.Cu at (97.5, 21.7)
- added C36: 100n, Capacitor_SMD:C_0603_1608Metric, F.Cu at (97.5, 24.2)
- added C37: 100n, Capacitor_SMD:C_0603_1608Metric, F.Cu at (97.5, 26.7)
- added C38: 100n, Capacitor_SMD:C_0603_1608Metric, F.Cu at (97.5, 29.2)
- added C39: 100n, Capacitor_SMD:C_0603_1608Metric, F.Cu at (101.5, 16.7)
- added C40: 100n, Capacitor_SMD:C_0603_1608Metric, F.Cu at (101.5, 19.2)
- added D10: 1N4148W-TP, Diode_SMD:D_SOD-123, F.Cu at (65.4, 33.9)
- added D11: 1N4148W-TP, Diode_SMD:D_SOD-123, F.Cu at (65.4, 37.2)
- added D12: 1N4148W-TP, Diode_SMD:D_SOD-123, F.Cu at (65.4, 40.6)
- added D13: 1N4148W-TP, Diode_SMD:D_SOD-123, F.Cu at (65.4, 43.9)
- added D14: 1N4148W-TP, Diode_SMD:D_SOD-123, F.Cu at (71.2, 17.1)
- added D15: 1N4148W-TP, Diode_SMD:D_SOD-123, F.Cu at (71.2, 20.5)
- added D16: 1N4148W-TP, Diode_SMD:D_SOD-123, F.Cu at (71.2, 23.8)
- added D17: 1N4148W-TP, Diode_SMD:D_SOD-123, F.Cu at (71.2, 27.2)
- added D19: 1N4148W-TP, Diode_SMD:D_SOD-123, F.Cu at (71.2, 30.5)
- added D20: 1N4148W-TP, Diode_SMD:D_SOD-123, F.Cu at (71.2, 33.9)
- added D21: 1N4148W-TP, Diode_SMD:D_SOD-123, F.Cu at (71.2, 37.2)
- added D22: 1N4148W-TP, Diode_SMD:D_SOD-123, F.Cu at (71.2, 40.6)
- added D23: 1N4148W-TP, Diode_SMD:D_SOD-123, F.Cu at (71.2, 43.9)
- added D24: 1N4148W-TP, Diode_SMD:D_SOD-123, F.Cu at (77.0, 17.1)
- added D25: 1N4148W-TP, Diode_SMD:D_SOD-123, F.Cu at (77.0, 20.5)
- added D26: 1N4148W-TP, Diode_SMD:D_SOD-123, F.Cu at (77.0, 23.8)
- added D27: 1N4148W-TP, Diode_SMD:D_SOD-123, F.Cu at (77.0, 27.2)
- added D28: 1N4148W-TP, Diode_SMD:D_SOD-123, F.Cu at (77.0, 30.5)
- added D29: 1N4148W-TP, Diode_SMD:D_SOD-123, F.Cu at (77.0, 33.9)
- added D30: 1N4148W-TP, Diode_SMD:D_SOD-123, F.Cu at (77.0, 37.2)
- added D31: 1N4148W-TP, Diode_SMD:D_SOD-123, F.Cu at (77.0, 40.6)
- added D32: 1N4148W-TP, Diode_SMD:D_SOD-123, F.Cu at (77.0, 43.9)
- added D33: 1N4148W-TP, Diode_SMD:D_SOD-123, F.Cu at (82.8, 17.1)
- added D34: 1N4148W-TP, Diode_SMD:D_SOD-123, F.Cu at (82.8, 20.5)
- added D35: 1N4148W-TP, Diode_SMD:D_SOD-123, F.Cu at (82.8, 23.8)
- added D36: 1N4148W-TP, Diode_SMD:D_SOD-123, F.Cu at (82.8, 27.2)
- added D37: 1N4148W-TP, Diode_SMD:D_SOD-123, F.Cu at (82.8, 30.5)
- added D38: 1N4148W-TP, Diode_SMD:D_SOD-123, F.Cu at (82.8, 33.9)
- added D39: 1N4148W-TP, Diode_SMD:D_SOD-123, F.Cu at (82.8, 37.2)
- added D4: 1N4148W-TP, Diode_SMD:D_SOD-123, F.Cu at (65.4, 17.1)
- added D40: 1N4148W-TP, Diode_SMD:D_SOD-123, F.Cu at (82.8, 40.6)
- added D41: 1N4148W-TP, Diode_SMD:D_SOD-123, F.Cu at (82.8, 43.9)
- added D42: 1N4148W-TP, Diode_SMD:D_SOD-123, F.Cu at (88.6, 17.1)
- added D43: 1N4148W-TP, Diode_SMD:D_SOD-123, F.Cu at (88.6, 20.5)
- added D44: 1N4148W-TP, Diode_SMD:D_SOD-123, F.Cu at (88.6, 23.8)
- added D45: 1N4148W-TP, Diode_SMD:D_SOD-123, F.Cu at (88.6, 27.2)
- added D46: 1N4148W-TP, Diode_SMD:D_SOD-123, F.Cu at (88.6, 30.5)
- added D47: 1N4148W-TP, Diode_SMD:D_SOD-123, F.Cu at (88.6, 33.9)
- added D48: 1N4148W-TP, Diode_SMD:D_SOD-123, F.Cu at (88.6, 37.2)
- added D49: 1N4148W-TP, Diode_SMD:D_SOD-123, F.Cu at (88.6, 40.6)
- added D5: 1N4148W-TP, Diode_SMD:D_SOD-123, F.Cu at (65.4, 20.5)
- added D6: 1N4148W-TP, Diode_SMD:D_SOD-123, F.Cu at (65.4, 23.8)
- added D8: 1N4148W-TP, Diode_SMD:D_SOD-123, F.Cu at (65.4, 27.2)
- added D9: 1N4148W-TP, Diode_SMD:D_SOD-123, F.Cu at (65.4, 30.5)
- added L1: 1u, ZF_common:XFL4020-102MEC, F.Cu at (80.4, 80.0)
- added R21: 1k, Resistor_SMD:R_0603_1608Metric, F.Cu at (58.1, 22.8)
- added R22: 1k, Resistor_SMD:R_0603_1608Metric, F.Cu at (58.1, 25.3)
- added R23: 1k, Resistor_SMD:R_0603_1608Metric, F.Cu at (101.5, 21.7)
- added R7: 620R, Resistor_SMD:R_0603_1608Metric, F.Cu at (91.5, 58.2)
- added SW2: SKRHABE010, ZF_common:SKRHABE010, F.Cu at (97.1, 36.3)
- added U3: RP2040, Package_DFN_QFN:QFN-56-1EP_7x7mm_P0.4mm_EP3.2x3.2mm, F.Cu at (96.1, 46.7)
- added U5: TS3USB221ERSER, ZF_common:TS3USB221ERSER, F.Cu at (37.5, 75.9)
- added Y1: X322512MSB4SI, Crystal:Crystal_SMD_3225-4Pin_3.2x2.5mm, F.Cu at (75.5, 47.9)
- C1, C5, C6: value 10u -> 100n
- C12, C13: value 47n -> 10u
- C14: value 100n -> 2u2
- C19, C20: value 10u -> 47n
- C2: value 22u -> 100n
- C21, C4, C8: value 100n -> 10u
- C23: value 10u -> 22u
- C3: value 4u7 -> 10u
- C7: value 2u2 -> 100n
- Q1: value CSD17575Q3 -> CSD17570Q5B
- R1: value 2 -> 2k2
- R10: value 10k -> 50R
- R11: value 2k2 -> 10k
- R12: value 100 -> 2R
- R15: value 1k -> 300k
- R16: value 1k -> 10k
- R17: value 10k -> 732k
- R19: value 732k -> 2k2
- R2, R9: value 10k -> 100R
- R20: value 620 -> 3k
- R24: value 15k -> 27R
- R25: value 100 -> 27R
- R3: value 3k -> 10k
- R5: value 300k -> 10k
- R6: value 2k2 -> 2k
- R8: value 2k -> 15k
- U1: value RP2040 -> BQ25792RQMR; footprint Package_DFN_QFN:QFN-56-1EP_7x7mm_P0.4mm_EP3.2x3.2mm -> ZF_common:BQ25792RQMR
- U2: value BQ25792RQMR -> TPS61022RWUR; footprint ZF_common:BQ25792RQMR -> Package_DFN_QFN:Texas_RWU0007A_VQFN-7_2x2mm_P0.5mm
- U4: value TPS61022 -> W25Q16JVSS; footprint Package_DFN_QFN:Texas_RWU0007A_VQFN-7_2x2mm_P0.5mm -> Package_SO:SOIC-8_5.3x5.3mm_P1.27mm
- moved C1 71.5 mm to (31.7, 74.8)
- moved C2 71.5 mm to (31.7, 77.3)
- moved R1 71.1 mm to (31.7, 79.8)
- moved R5 58.3 mm to (87.5, 75.8)
- moved C10 55.8 mm to (79.5, 73.3)
- moved C11 55.8 mm to (79.5, 75.8)
- moved C19 55.8 mm to (83.5, 73.3)
- moved C20 55.8 mm to (83.5, 75.8)
- moved J12401826E412A1 49.8 mm to (20.6, 79.5)
- moved L2 48.0 mm to (80.4, 85.8)
- moved R20 46.0 mm to (95.5, 68.2)
- moved R18 46.0 mm to (95.5, 63.2)
- moved R19 46.0 mm to (95.5, 65.7)
- moved D1 44.2 mm to (64.8, 84.9)
- moved R14 41.0 mm to (91.5, 75.8)
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Connections:
- net /Base/USB3_RX1_N renamed /USB-C/USB3_RX1_N
- net /Base/USB3_RX1_P renamed /USB-C/USB3_RX1_P
- net /Base/USB3_RX2_N renamed /USB-C/USB3_RX2_N
- net /Base/USB3_RX2_P renamed /USB-C/USB3_RX2_P
- net /Base/USB3_TX1_N renamed /USB-C/USB3_TX1_N
- net /Base/USB3_TX1_P renamed /USB-C/USB3_TX1_P
- net /Base/USB3_TX2_N renamed /USB-C/USB3_TX2_N
- net /Base/USB3_TX2_P renamed /USB-C/USB3_TX2_P
- C1 pad 1: /Base/Power Management/VSYS -> /Power Management/VBUS
- C10 pad 1: Net-(U2-PMID) -> /Power Management/VSYS
- C11 pad 1: Net-(U2-PMID) -> /Power Management/VBUS
- C12 pad 1: /Base/Power Management/SW2 -> Net-(U1-PMID)
- C12 pad 2: /Base/Power Management/BTST2 -> GND
- C13 pad 1: /Base/Power Management/BTST1 -> /Power Management/VSYS
- C13 pad 2: /Base/Power Management/SW1 -> GND
- C14 pad 1: /Base/Power Management/VSYS -> Net-(C14-Pad1)
- C15 pad 1: /Base/Power Management/VSYS -> Net-(U1-PMID)
- C16 pad 1: /Base/Power Management/VSYS -> /Power Management/VSYS
- C17 pad 1: /Base/Power Management/VSYS -> /Power Management/VSYS
- C18 pad 1: /Base/Power Management/VSYS -> /Power Management/VSYS
- C19 pad 1: /Base/Power Management/VSYS -> /Power Management/BTST1
- C19 pad 2: GND -> /Power Management/SW1
- C2 pad 1: +5V -> /Power Management/VBUS
- C20 pad 1: /Base/Power Management/BAT -> /Power Management/SW2
- C20 pad 2: GND -> /Power Management/BTST2
- C21 pad 1: +5V -> /Power Management/VSYS
- C23 pad 1: /Base/Power Management/BAT -> /CM5 GPIO/+5v
- C24 pad 1: +5V -> /CM5 GPIO/+5v
- C25 pad 1: +5V -> /CM5 GPIO/+5v
- C26 pad 1: +5V -> /CM5 GPIO/+3.3v
- C3 pad 1: /Base/Power Management/REGN -> /Power Management/BAT
- C4 pad 1: VBUS -> /Power Management/BAT
- C5 pad 1: VBUS -> /Power Management/VBUS
- C6 pad 1: VBUS -> Net-(U1-PMID)
- C7 pad 1: Net-(C7-Pad1) -> /Power Management/VSYS
- C8 pad 1: Net-(U2-PMID) -> /Power Management/VBUS
- C9 pad 1: Net-(U2-PMID) -> Net-(U1-PMID)
- D1 pad 1: /Base/Power Management/STAT -> /Power Management/STAT
- D2 pad 2: +3V3 -> /CM5 GPIO/+3.3v
- D3 pad 2: +3V3 -> /CM5 GPIO/+3.3v
- J1 pad 2: /Base/Power Management/BATT_TEMP -> /Power Management/BATT_TEMP
- J12401826E412A1 pad A4: VBUS -> /Power Management/VBUS
- J12401826E412A1 pad A5: /Base/CC1 -> /CM5 GPIO/CC1
- J12401826E412A1 pad A6: /Base/USB2_P -> /CM5 Highspeed/USB2_P
- J12401826E412A1 pad A7: /Base/USB2_N -> /CM5 Highspeed/USB2_N
- J12401826E412A1 pad A9: VBUS -> /Power Management/VBUS
- J12401826E412A1 pad B4: VBUS -> /Power Management/VBUS
- J12401826E412A1 pad B5: /Base/CC2 -> /CM5 GPIO/CC2
- J12401826E412A1 pad B6: /Base/USB2_P -> /CM5 Highspeed/USB2_P
- J12401826E412A1 pad B7: /Base/USB2_N -> /CM5 Highspeed/USB2_N
- J12401826E412A1 pad B9: VBUS -> /Power Management/VBUS
- J2 pad 2: /Base/Power Management/BATT_TEMP -> /Power Management/BATT_TEMP
- L2 pad 1: /Base/Power Management/VSYS -> /Power Management/SW1
- L2 pad 2: Net-(U4-SW) -> /Power Management/SW2
- Module1 pad 21: /Base/CM5 GPIO/LED_nACT -> /CM5 GPIO/LED_nACT
- Module1 pad 54: unconnected-(Module1A-GPIO4-Pad54) -> /CM5 GPIO/SWCLK
- Module1 pad 56: unconnected-(Module1A-GPIO3-Pad56) -> /CM5 GPIO/SWD
- Module1 pad 58: unconnected-(Module1A-GPIO2-Pad58) -> /CM5 GPIO/PMIC_INT
- Module1 pad 77: unconnected-(Module1A-+5v_(Input)-Pad77) -> /CM5 GPIO/+5v
- Module1 pad 79: unconnected-(Module1A-+5v_(Input)-Pad79) -> /CM5 GPIO/+5v
- Module1 pad 81: unconnected-(Module1A-+5v_(Input)-Pad81) -> /CM5 GPIO/+5v
- Module1 pad 83: unconnected-(Module1A-+5v_(Input)-Pad83) -> /CM5 GPIO/+5v
- Module1 pad 84: unconnected-(Module1A-+3.3v_(Output)-Pad84) -> /CM5 GPIO/+3.3v
- Module1 pad 85: unconnected-(Module1A-+5v_(Input)-Pad85) -> /CM5 GPIO/+5v
- Module1 pad 86: unconnected-(Module1A-+3.3v_(Output)-Pad86) -> /CM5 GPIO/+3.3v
- Module1 pad 87: unconnected-(Module1A-+5v_(Input)-Pad87) -> /CM5 GPIO/+5v
- Module1 pad 92: PWR_BUT -> /Power Management/QON
- Module1 pad 94: unconnected-(Module1A-CC1-Pad94) -> /CM5 GPIO/CC1
- Module1 pad 95: /Base/CM5 GPIO/LED_nPWR -> /CM5 GPIO/LED_nPWR
- Module1 pad 96: unconnected-(Module1A-CC2-Pad96) -> /CM5 GPIO/CC2
- Q1 pad 4: /Base/Power Management/SDRV -> /Power Management/SDRV
- Q1 pad 5: /Base/Power Management/BAT -> /Power Management/BAT
- R1 pad 1: VBUS -> /Power Management/VBUS
- R1 pad 2: Net-(C7-Pad1) -> GND
- R10 pad 1: Net-(U2-SDA) -> Net-(R10-Pad1)
- R10 pad 2: /Base/Power Management/SDA -> GND
- R11 pad 1: VBUS -> /CM5 GPIO/PMIC_INT
- R11 pad 2: GND -> Net-(U1-~{INT})
- R12 pad 1: V_BATT -> /Power Management/VBUS
- R12 pad 2: /Base/Power Management/BATP -> Net-(C14-Pad1)
- R13 pad 1: /Base/Power Management/INT -> /Power Management/VSYS
- R13 pad 2: Net-(U2-~{INT}) -> Net-(U2-EN)
- R14 pad 1: /Base/Power Management/REGN -> /Power Management/REGN
- R14 pad 2: /Base/Power Management/ILIM_HIZ -> /Power Management/ILIM_HIZ
- R15 pad 1: Net-(D2-K) -> /Power Management/ILIM_HIZ
- R15 pad 2: /Base/CM5 GPIO/LED_nPWR -> GND
- R16 pad 1: Net-(D3-K) -> /Power Management/REGN
- R16 pad 2: /Base/CM5 GPIO/LED_nACT -> /Power Management/QON
- R17 pad 1: /Base/Power Management/VSYS -> /CM5 GPIO/+5v
- R17 pad 2: Net-(U4-EN) -> Net-(U2-FB)
- R18 pad 1: Net-(U4-FB) -> Net-(U2-FB)
- R19 pad 1: +5V -> /Power Management/REGN
- R19 pad 2: Net-(U4-FB) -> Net-(D1-A)
- R2 pad 1: GND -> /Power Management/BATP
- R2 pad 2: Net-(U2-~{CE}) -> V_BATT
- R20 pad 1: Net-(R20-Pad1) -> /Power Management/PROG
- R20 pad 2: /Base/Power Management/BATT_TEMP -> GND
- R24 pad 1: /Base/Power Management/BATT_TEMP -> unconnected-(R24-Pad1)
- R24 pad 2: Net-(R24-Pad2) -> /Keyboard/USB_DP
- R25 pad 1: Net-(R24-Pad2) -> unconnected-(R25-Pad1)
- R25 pad 2: Net-(R25-Pad2) -> /Keyboard/USB_DN
- R3 pad 1: Net-(U2-PROG) -> unconnected-(R3-Pad1)
- R3 pad 2: GND -> /Power Management/SCL
- R4 pad 1: /Base/Power Management/REGN -> /Power Management/SDA
- R4 pad 2: PWR_BUT -> unconnected-(R4-Pad2)
- R5 pad 1: /Base/Power Management/ILIM_HIZ -> GND
- R5 pad 2: GND -> Net-(U1-~{CE})
- R6 pad 1: /Base/Power Management/REGN -> /Power Management/REGN
- R6 pad 2: Net-(D1-A) -> Net-(R6-Pad2)
- R8 pad 1: /Base/Power Management/REGN -> /Power Management/BATT_TEMP
- R8 pad 2: Net-(R20-Pad1) -> Net-(R8-Pad2)
- R9 pad 1: /Base/Power Management/SCL -> Net-(R8-Pad2)
- R9 pad 2: Net-(U2-SCL) -> Net-(R10-Pad1)
- U1 pad 1: Net-(U1-IOVDD-Pad1) -> /Power Management/STAT
- U1 pad 10: Net-(U1-IOVDD-Pad1) -> GND
- U1 pad 11: unconnected-(U1-GPIO8-Pad11) -> GND
- U1 pad 12: unconnected-(U1-GPIO9-Pad12) -> /Power Management/QON
- U1 pad 13: unconnected-(U1-GPIO10-Pad13) -> Net-(U1-~{CE})
- U1 pad 14: unconnected-(U1-GPIO11-Pad14) -> /Power Management/SCL
- U1 pad 15: unconnected-(U1-GPIO12-Pad15) -> /Power Management/SDA
- U1 pad 16: unconnected-(U1-GPIO13-Pad16) -> /Power Management/BATT_TEMP
- U1 pad 17: unconnected-(U1-GPIO14-Pad17) -> /Power Management/ILIM_HIZ
- U1 pad 18: unconnected-(U1-GPIO15-Pad18) -> /Power Management/BATP
- U1 pad 19: unconnected-(U1-TESTEN-Pad19) -> /Power Management/BTST2
- U1 pad 2: unconnected-(U1-GPIO0-Pad2) -> /Power Management/VBUS
- U1 pad 20: unconnected-(U1-XIN-Pad20) -> /Power Management/PROG
- U1 pad 21: unconnected-(U1-XOUT-Pad21) -> Net-(U1-~{INT})
- U1 pad 22: Net-(U1-IOVDD-Pad1) -> /Power Management/BAT
- U1 pad 23: Net-(U1-DVDD-Pad23) -> /Power Management/BAT
- U1 pad 24: unconnected-(U1-SWCLK-Pad24) -> /Power Management/SDRV
- U1 pad 25: unconnected-(U1-SWD-Pad25) -> /Power Management/VSYS
- U1 pad 26: unconnected-(U1-RUN-Pad26) -> /Power Management/SW2
- U1 pad 27: unconnected-(U1-GPIO16-Pad27) -> GND
- U1 pad 28: unconnected-(U1-GPIO17-Pad28) -> /Power Management/SW1
- U1 pad 29: unconnected-(U1-GPIO18-Pad29) -> Net-(U1-PMID)
- U1 pad 3: unconnected-(U1-GPIO1-Pad3) -> /Power Management/VBUS
- U1 pad 4: unconnected-(U1-GPIO2-Pad4) -> /Power Management/BTST1
- U1 pad 5: unconnected-(U1-GPIO3-Pad5) -> /Power Management/REGN
- U1 pad 6: unconnected-(U1-GPIO4-Pad6) -> /CM5 Highspeed/USB2_P
- U1 pad 7: unconnected-(U1-GPIO5-Pad7) -> /CM5 Highspeed/USB2_N
- U1 pad 8: unconnected-(U1-GPIO6-Pad8) -> /Power Management/VBUS
- U1 pad 9: unconnected-(U1-GPIO7-Pad9) -> /Power Management/VBUS
- U2 pad 1: /Base/Power Management/STAT -> GND
- U2 pad 2: VBUS -> Net-(U2-SW)
- U2 pad 3: VBUS -> /CM5 GPIO/+5v
- U2 pad 4: /Base/Power Management/BTST1 -> Net-(U2-FB)
- U2 pad 5: /Base/Power Management/REGN -> Net-(U2-EN)
- U2 pad 6: /Base/USB2_P -> Net-(U2-EN)
- U2 pad 7: /Base/USB2_N -> /Power Management/VSYS
- U4 pad 1: GND -> /Keyboard/CS
- U4 pad 2: Net-(U4-SW) -> /Keyboard/SD1
- U4 pad 3: +5V -> /Keyboard/SD2
- U4 pad 4: Net-(U4-FB) -> GND
- U4 pad 5: Net-(U4-EN) -> /Keyboard/SD0
- U4 pad 6: Net-(U4-EN) -> /Keyboard/SD_CLK
- U4 pad 7: /Base/Power Management/VSYS -> /Keyboard/SD3
